File: TP_DCI_Gustavo_Paredes/EjercicioGustavoParedes/EjercicioGustavoParedes.sch (KiCad schematic (older format))
At the start: 5 parts, among them J1 Conn_01x03

Commit message: 1er Version
Primera version del ejercicio aulico.
Parts:
- C1: footprint Capacitor_SMD:C_0603_1608Metric -> Capacitor_THT:CP_Radial_D4.0mm_P2.00mm
- D1: footprint Diode_SMD:D_SOD-323 -> LED_THT:LED_D3.0mm
- D2: footprint Diode_SMD:D_SOD-323 -> Diode_THT:D_5W_P10.16mm_Horizontal; symbol Simulation_SPICE:DIODE -> EjercicioGustavoParedes-rescue:DIODE-Simulation_SPICE
- J1: footprint Diode_SMD:D_SOD-323 -> Connector_PinHeader_1.00mm:PinHeader_1x03_P1.00mm_Vertical
- R1: footprint Resistor_SMD:R_0603_1608Metric -> Resistor_THT:R_Axial_DIN0204_L3.6mm_D1.6mm_P1.90mm_Vertical
Changed lines of the file:
@@
 EESchema Schematic File Version 4
-EELAYER 29 0
+LIBS:EjercicioGustavoParedes-cache
+EELAYER 26 0
 EELAYER END
 $Descr A4 11693 8268
@@
 F 0 "C1" V 3552 1700 50  0000 C CNN
 F 1 "100nF" V 3461 1700 50  0000 C CNN
-F 2 "Capacitor_SMD:C_0603_1608Metric" H 3338 1550 50  0001 C CNN
+F 2 "Capacitor_THT:CP_Radial_D4.0mm_P2.00mm" H 3338 1550 50  0001 C CNN
 F 3 "~" H 3300 1700 50  0001 C CNN
 	1    3300 1700
@@
 F 0 "J1" H 2468 2117 50  0000 C CNN
 F 1 "Conn_01x03" H 2468 2026 50  0000 C CNN
-F 2 "Diode_SMD:D_SOD-323" H 2550 1800 50  0001 C CNN
+F 2 "Connector_PinHeader_1.00mm:PinHeader_1x03_P1.00mm_Vertical" H 2550 1800 50  0001 C CNN
 F 3 "~" H 2550 1800 50  0001 C CNN
 	1    2550 1800
@@
 F 0 "D1" H 3293 1266 50  0000 C CNN
 F 1 "LED" H 3293 1175 50  0000 C CNN
-F 2 "Diode_SMD:D_SOD-323" H 3300 1050 50  0001 C CNN
+F 2 "LED_THT:LED_D3.0mm" H 3300 1050 50  0001 C CNN
 F 3 "~" H 3300 1050 50  0001 C CNN
 	1    3300 1050
@@
 $EndComp
 $Comp
-L Simulation_SPICE:DIODE D2
+L EjercicioGustavoParedes-rescue:DIODE-Simulation_SPICE D2
 U 1 1 5CE4B87C
 P 3300 2250
 F 0 "D2" H 3300 2467 50  0000 C CNN
 F 1 "1N4148" H 3300 2376 50  0000 C CNN
-F 2 "Diode_SMD:D_SOD-323" H 3300 2250 50  0001 C CNN
+F 2 "Diode_THT:D_5W_P10.16mm_Horizontal" H 3300 2250 50  0001 C CNN
 F 3 "~" H 3300 2250 50  0001 C CNN
 F 4 "Y" H 3300 2250 50  0001 L CNN "Spice_Netlist_Enabled"
@@
 F 0 "R1" H 3820 2046 50  0000 L CNN
 F 1 "100k" H 3820 1955 50  0000 L CNN
-F 2 "Resistor_SMD:R_0603_1608Metric" V 3680 2000 50  0001 C CNN
+F 2 "Resistor_THT:R_Axial_DIN0204_L3.6mm_D1.6mm_P1.90mm_Vertical" V 3680 2000 50  0001 C CNN
 F 3 "~" H 3750 2000 50  0001 C CNN
 	1    3750 2000
@@
 Wire Wire Line
 	2950 1050 2950 1700
-Connection ~ 2950 1700
-Wire Wire Line
-	2950 1700 2750 1700
 Wire Wire Line
 	3450 1050 3750 1050
@@
 Wire Wire Line
 	2950 2250 2950 1900
-Wire Wire Line
-	2950 1900 2750 1900
 NoConn ~ 2750 1800
 Text Notes 4450 1550 0    50   ~ 0
 R Serie
+Wire Wire Line
+	2950 1900 2750 1900
+Wire Wire Line
+	2750 1700 2950 1700
+Connection ~ 2950 1700
 $EndSCHEMATC
